File: hardware/pcb/smart_plants_breakout_ws-board_rev1/smart_plants_breakout_ws-board_rev1.kicad_pcb (KiCad board)
At the start: 2 copper layers, 48.3 x 48.3 mm, 27 parts, among them J1 Conn_01x09_Pin, J10 Pump, J11 I2C D3-powered, J2 Conn_01x09_Pin, J3 I2C, J4 USB-C Power, J5 I2C D2-powered, J6 I2C, J7 Battery, J9 Moisture Sensor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

Commit message: WS PCB bug fixes
Parts:
- J4: footprint Connector_JST:JST_XH_B2B-XH-A_1x02_P2.50mm_Vertical -> Connector_JST:JST_PH_B2B-PH-K_1x02_P2.00mm_Vertical
Connections:
- J10 pad 1: Net-(D1-A) -> Net-(D1-K)
- J10 pad 2: Net-(D1-K) -> Net-(D1-A)
- J9 pad 2: VDC -> Net-(J2-Pin_8)
Routing:
- net Net-(J2-Pin_8): track 4.45 -> 35.4 mm
- net VDC: track 86.4 -> 101.7 mm
- net Net-(D1-A): track 40.2 -> 47.1 mm
- net Net-(D1-K): track 97.3 -> 98.4 mm
